Commit message: modified kuka link mass, moment of inertia and damping according to CAD model, the torque bias still exists, need further diagnosis

File: drake/examples/kuka_iiwa_arm/urdf/iiwa14_old.urdf (robot description, URDF)
Before this commit: robot iiwa14, 11 links, 10 joints
Links:
- link iiwa_link_1: mass 5.76 -> 4
- link iiwa_link_2: mass 3.95 -> 4
- link iiwa_link_3: mass 3.18 -> 3
- link iiwa_link_4: mass 2.74 -> 2.7
- link iiwa_link_5: mass 1.69 -> 1.7
- link iiwa_link_7: mass 0.31 -> 0.3
