Commit message: (i) update the urdf mass and moment of inertia according to gravity comp torque comparison test, (ii) add an inverse dynamics test, to be debugged

File: drake/examples/kuka_iiwa_arm/urdf/iiwa14.urdf (robot description, URDF)
Before this commit: robot iiwa14, 11 links, 10 joints
Links:
- link iiwa_link_2: mass 3.95 -> 6.35
- link iiwa_link_3: mass 3.18 -> 3.5
- link iiwa_link_4: mass 2.74 -> 3.5
- link iiwa_link_5: mass 1.69 -> 3.5
- link iiwa_link_7: mass 0.31 -> 1.2
