Commit message: Variational traj opt working for HAMR, but is slow. Note that RigidBodyLoop stiffness/damping works for HAMR, but might not work near singularities in euler angles

File: drake/examples/HAMR-URDF/urdf/HAMRVariational_scaled.urdf (robot description, URDF)
Before this commit: robot Hamr, 28 links, 24 joints
Links:
- added link FRL1, mass 4.5174E-03; visual mesh filename=../meshes/FRL1.obj scale=1000
- added link FRL2, mass 1.6211E-03; visual mesh filename=../meshes/FRL2.obj scale=1000
- added link FRL3, mass 4.2308E-03; visual mesh filename=../meshes/FRL3.obj scale=1000
- added link FRL4, mass 6.9770e-03; visual mesh filename=../meshes/FRL4.obj scale=1000
- added link FRLeg, mass 1.6993E-02; collision sphere radius=0; visual mesh filename=../meshes/FRLeg.obj scale=1000
- added link FRS1, mass 8.9854E-04; visual mesh filename=../meshes/FRS1.obj scale=1000
- added link FRS2, mass 7.2648E-03; visual mesh filename=../meshes/FRS2.obj scale=1000
- added link FRS3, mass 3.889E-03; visual mesh filename=../meshes/FRS3.obj scale=1000
- added link FRS4, mass 1.4269E-02; visual mesh filename=../meshes/FRS4.obj scale=1000
- added link RRL1, mass 3.4357E-03; visual mesh filename=../meshes/RRL1.obj scale=1000
- added link RRL2, mass 1.6211E-03; visual mesh filename=../meshes/RRL2.obj scale=1000
- added link RRL3, mass 4.2308E-03; visual mesh filename=../meshes/RRL3.obj scale=1000
- added link RRL4, mass 6.9770e-03; visual mesh filename=../meshes/RRL4.obj scale=1000
- added link RRL_Loop, mass 0.1286; visual mesh filename=../meshes/Chassis.obj scale=1000
- added link RRLeg, mass 1.6993E-02; collision sphere radius=0; visual mesh filename=../meshes/FRLeg.obj scale=1000
- added link RRS1, mass 8.9854E-04; visual mesh filename=../meshes/RRS1.obj scale=1000
- added link RRS2, mass 7.2648E-03; visual mesh filename=../meshes/RRS2.obj scale=1000
- added link RRS3, mass 3.889E-03; visual mesh filename=../meshes/RRS3.obj scale=1000
- added link RRS4, mass 1.4269E-02; visual mesh filename=../meshes/RRS4.obj scale=1000
- added link RRSFB_Loop, mass 6.9770e-03; visual mesh filename=../meshes/RRL4.obj scale=1000
- added link RRS_Loop, mass 0.1286; visual mesh filename=../meshes/Chassis.obj scale=1000
- link FRSFB_Loop: geometry visual mesh filename=../meshes/FRL4.obj scale=1000
Joints:
- added joint FRLegJoint: type fixed, parent FRL4, child FRLeg, origin xyz=6E-02 -4.64367405164 -4.80326038678 rpy=0 0 0, axis 0 0 0
- added joint FRqfb1: type revolute, parent FRS3, child FRS4, origin xyz=1.52236486487 -0.12 -1.25 rpy=0 0 0, axis 1 0 0, limit lower=-pi/3 upper=pi/3
- added joint FRqfb2: type continuous, parent FRS4, child FRSFB_Loop, origin xyz=-2.05236472111 -5.98079552649 0.0 rpy=0 0 0, axis 0 1 0, limit lower=-pi/3 upper=pi/3
- added joint FRqfb3: type revolute, parent FRL3, child FRL4, origin xyz=2.25 -0.12 -1.07 rpy=0 0 0, axis 0 0 1, limit lower=-pi/3 upper=pi/3
- added joint FRql1: type revolute, parent FRL1, child FRL2, origin xyz=0 -4.57322017852 0.38168853124 rpy=0 0 0, axis 1 0 0, limit lower=-pi/3 upper=pi/3
- added joint FRql2: type revolute, parent FRL2, child FRL3, origin xyz=0 -1.945 0 rpy=0 0 0, axis 1 0 0, limit lower=-pi/3 upper=pi/3
- added joint FRql3: type continuous, parent FRL3, child FRL_Loop, origin xyz=0.0, -0.12, 0.58 rpy=0 0 0, axis 1 0 0, limit lower=-pi/3 upper=pi/3
- added joint FRqlact: type prismatic, parent Chassis, child FRL1, origin xyz=10.504659815390 -3.151779821480 -0.501688531240 rpy=0 0 0, axis 0 1 0
- added joint FRqs1: type revolute, parent FRS1, child FRS2, origin xyz=0 -0.77116874934 0.12648211488 rpy=0 0 0, axis 0 0 1, limit lower=-pi/3 upper=pi/3
- added joint FRqs2: type revolute, parent FRS2, child FRS3, origin xyz=0 -7.44214712409 2.06176831433 rpy=0 0 0, axis 0 0 1, limit lower=-pi/3 upper=pi/3
- added joint FRqs3: type continuous, parent FRS3, child FRS_Loop, origin xyz=-0.53, -0.12, 0.0 rpy=0 0 0, axis 0 0 1, limit lower=-pi/3 upper=pi/3
- added joint FRqsact: type prismatic, parent Chassis, child FRS1, origin xyz=13.284659815390 -1.456684126580 -0.478250429210 rpy=0 0 0, axis 0 1 0
- added joint RRLegJoint: type Fixed, parent RRL4, child RRLeg, origin xyz=-6E-02 -4.64367405164 -4.80326038678 rpy=0 0 0, axis 0 0 0
- added joint RRqfb1: type revolute, parent RRS3, child RRS4, origin xyz=-1.52236486487 -0.12 -1.25 rpy=0 0 0, axis 1 0 0, limit lower=-pi/3 upper=pi/3
- added joint RRqfb2: type continuous, parent RRS4, child RRSFB_Loop, origin xyz=2.05236472111 -5.98079552649 0.0 rpy=0 0 0, axis 0 1 0, limit lower=-pi/3 upper=pi/3
- added joint RRqfb3: type revolute, parent RRL3, child RRL4, origin xyz=-2.25 -0.12 -1.07 rpy=0 0 0, axis 0 0 1, limit lower=-pi/3 upper=pi/3
- added joint RRql1: type revolute, parent RRL1, child RRL2, origin xyz=0 -2.93322017852 0.38168853124 rpy=0 0 0, axis 1 0 0, limit lower=-pi/3 upper=pi/3
- added joint RRql2: type revolute, parent RRL2, child RRL3, origin xyz=0 -1.945 0 rpy=0 0 0, axis 1 0 0, limit lower=-pi/3 upper=pi/3
- added joint RRql3: type continuous, parent RRL3, child RRL_Loop, origin xyz=0.0, -0.12, 0.58 rpy=0 0 0, axis 1 0 0, limit lower=-pi/3 upper=pi/3
- added joint RRqlact: type prismatic, parent Chassis, child RRL1, origin xyz=-10.504659815390 -4.791779821480 -0.501688531240 rpy=0 0 0, axis 0 1 0
- added joint RRqs1: type revolute, parent RRS1, child RRS2, origin xyz=0 -0.77116874934 0.12648211488 rpy=0 0 0, axis 0 0 1, limit lower=-pi/3 upper=pi/3
- added joint RRqs2: type revolute, parent RRS2, child RRS3, origin xyz=0 -7.44214712409 2.06176831433 rpy=0 0 0, axis 0 0 1, limit lower=-pi/3 upper=pi/3
- added joint RRqs3: type continuous, parent RRS3, child RRS_Loop, origin xyz=0.53, -0.12, 0.0 rpy=0 0 0, axis 0 0 1, limit lower=-pi/3 upper=pi/3
- added joint RRqsact: type prismatic, parent Chassis, child RRS1, origin xyz=-13.284659815390 -1.456684126580 -0.478250429210 rpy=0 0 0, axis 0 1 0
- joint FLqlact: limit lower=-0.7 upper=0.7 -> (none)
- joint FLqsact: limit lower=-0.7 upper=0.7 -> (none)
- joint RLqlact: limit lower=-0.7 upper=0.7 -> (none)
- joint RLqsact: limit lower=-0.7 upper=0.7 -> (none)
