Commit message: Small changes to HAMR model to work better w/ traj opt

File: drake/examples/HAMR-URDF/urdf/HAMRVariational_scaledV2_LB.urdf (robot description, URDF)
Before this commit: robot Hamr, 49 links, 48 joints
Joints:
- joint FLql3: limit lower=-pi/3 upper=pi/4 -> lower=-pi/3 upper=pi/3
- joint FLqlact: limit (none) -> lower=-0.16 upper=0.3
- joint FLqsact: limit (none) -> lower=-0.3 upper=0.3
- joint FRqlact: limit (none) -> lower=-0.3 upper=0.16
- joint FRqsact: limit (none) -> lower=-0.3 upper=0.3
- joint RLqlact: limit (none) -> lower=-0.16 upper=0.3
- joint RLqsact: limit (none) -> lower=-0.3 upper=0.3
- joint RRqlact: limit (none) -> lower=-0.3 upper=0.16
- joint RRqsact: limit (none) -> lower=-0.3 upper=0.3

Commit message: tightened up joint limits further

File: drake/examples/HAMR-URDF/urdf/HAMRVariational_scaledV2_LB.urdf (robot description, URDF)
Before this commit: robot Hamr, 49 links, 48 joints
Joints:
- joint FLqlact: limit lower=-0.16 upper=0.3 -> lower=-0.16 upper=0.2
- joint FLqsact: limit lower=-0.3 upper=0.3 -> lower=-0.2 upper=0.2
- joint FRqlact: limit lower=-0.3 upper=0.16 -> lower=-0.2 upper=0.16
- joint FRqsact: limit lower=-0.3 upper=0.3 -> lower=-0.2 upper=0.2
- joint RLqlact: limit lower=-0.16 upper=0.3 -> lower=-0.16 upper=0.2
- joint RLqsact: limit lower=-0.3 upper=0.3 -> lower=-0.2 upper=0.2
- joint RRqlact: limit lower=-0.3 upper=0.16 -> lower=-0.2 upper=0.16
- joint RRqsact: limit lower=-0.3 upper=0.3 -> lower=-0.2 upper=0.2
