Commit message: fixed small bug with HAMR model

File: drake/examples/HAMR-URDF/urdf/HAMRVariational_scaledV2.urdf (robot description, URDF)
Before this commit: robot Hamr, 49 links, 48 joints
Links:
- link FRSFB_Loop: mass 1.4269E-02 -> 7.1345e-03

Commit message: Going back to a running traj-opt w/o pre-loaded lifts.

File: drake/examples/HAMR-URDF/urdf/HAMRVariational_scaledV2.urdf (robot description, URDF)
Before this commit: robot Hamr, 49 links, 48 joints
Links:
- link Chassis: mass 1.15747214880841 ->  1.2066
Joints:
- joint FLqlact: limit (none) -> lower=-0.2 upper=0.2
- joint FLqsact: limit (none) -> lower=-0.2 upper=0.2
- joint FRqlact: limit (none) -> lower=-0.2 upper=0.2
- joint FRqsact: limit (none) -> lower=-0.2 upper=0.2
- joint RLqlact: limit (none) -> lower=-0.2 upper=0.2
- joint RLqsact: limit (none) -> lower=-0.2 upper=0.2
- joint RRqlact: limit (none) -> lower=-0.2 upper=0.2
- joint RRqsact: limit (none) -> lower=-0.2 upper=0.2

Commit message: Prismatic Springs
added and tested RigidBodyPrismaticSpring class, using this for prismatic springs on HAMR instead of RigidBodySpringDamper b/c it's faster

File: drake/examples/HAMR-URDF/urdf/HAMRVariational_scaledV2.urdf (robot description, URDF)
Before this commit: robot Hamr, 49 links, 48 joints
Joints:
- joint FLqlact: limit lower=-0.2 upper=0.2 -> lower=-0.25 upper=0.25
- joint FLqsact: limit lower=-0.2 upper=0.2 -> lower=-0.25 upper=0.25
- joint FRqlact: limit lower=-0.2 upper=0.2 -> lower=-0.25 upper=0.25
- joint FRqsact: limit lower=-0.2 upper=0.2 -> lower=-0.25 upper=0.25
- joint RLqlact: limit lower=-0.2 upper=0.2 -> lower=-0.25 upper=0.25
- joint RLqsact: limit lower=-0.2 upper=0.2 -> lower=-0.25 upper=0.25
- joint RRqlact: limit lower=-0.2 upper=0.2 -> lower=-0.25 upper=0.25
- joint RRqsact: limit lower=-0.2 upper=0.2 -> lower=-0.25 upper=0.25
