Commit message: Cleaned up paths, improved fitting
now fitting on leg position as opposed to angle

File: drake/examples/HAMR-URDF/urdf/FL_scaled.urdf (robot description, URDF)
Before this commit: robot FrontLeftSingleLeg, 9 links, 8 joints
Links:
- link Chassis: geometry visual mesh filename=../meshes/Chassis.obj scale=1000
- link FLL1: geometry visual mesh filename=../meshes/FLL1.obj scale=1000
- link FLL2: geometry visual mesh filename=../meshes/FLL2.obj scale=1000
- link FLL3: geometry visual mesh filename=../meshes/FLL3.obj scale=1000
- link FLL4: geometry collision sphere radius=0; visual mesh filename=../meshes/FLL4.obj scale=1000
- link FLS1: geometry visual mesh filename=../meshes/FLS1.obj scale=1000
- link FLS2: geometry visual mesh filename=../meshes/FLS2.obj scale=1000
- link FLS3: geometry visual mesh filename=../meshes/FLS3.obj scale=1000
- link FLS4: geometry visual mesh filename=../meshes/FLS4.obj scale=1000

File: drake/examples/HAMR-URDF/urdf/FR_scaled.urdf (robot description, URDF)
Before this commit: robot FrontRightSingleLeg, 9 links, 8 joints
Links:
- link Chassis: geometry visual mesh filename=../meshes/Chassis.obj scale=1000
- link FRL1: geometry visual mesh filename=../meshes/FRL1.obj scale=1000
- link FRL2: geometry visual mesh filename=../meshes/FRL2.obj scale=1000
- link FRL3: geometry visual mesh filename=../meshes/FRL3.obj scale=1000
- link FRL4: geometry collision sphere radius=0; visual mesh filename=../meshes/FRL4.obj scale=1000
- link FRS1: geometry visual mesh filename=../meshes/FRS1.obj scale=1000
- link FRS2: geometry visual mesh filename=../meshes/FRS2.obj scale=1000
- link FRS3: geometry visual mesh filename=../meshes/FRS3.obj scale=1000
- link FRS4: geometry visual mesh filename=../meshes/FRS4.obj scale=1000

File: drake/examples/HAMR-URDF/urdf/HAMRSimple_scaled.urdf (robot description, URDF)
Before this commit: robot Hamr, 9 links, 8 joints
Links:
- link Chassis: geometry visual mesh filename=../meshes/Chassis.obj scale=1000

File: drake/examples/HAMR-URDF/urdf/RL_scaled.urdf (robot description, URDF)
Before this commit: robot RearLeftSingleLeg, 9 links, 8 joints
Links:
- link Chassis: geometry visual mesh filename=../meshes/Chassis.obj scale=1000
- link RLL1: geometry visual mesh filename=../meshes/RLL1.obj scale=1000
- link RLL2: geometry visual mesh filename=../meshes/RLL2.obj scale=1000
- link RLL3: geometry visual mesh filename=../meshes/RLL3.obj scale=1000
- link RLL4: geometry collision sphere radius=0; visual mesh filename=../meshes/RLL4.obj scale=1000
- link RLS1: geometry visual mesh filename=../meshes/RLS1.obj scale=1000
- link RLS2: geometry visual mesh filename=../meshes/RLS2.obj scale=1000
- link RLS3: geometry visual mesh filename=../meshes/RLS3.obj scale=1000
- link RLS4: geometry visual mesh filename=../meshes/RLS4.obj scale=1000

File: drake/examples/HAMR-URDF/urdf/RR_scaled.urdf (robot description, URDF)
Before this commit: robot RearRightSingleLeg, 9 links, 8 joints
Links:
- link Chassis: geometry visual mesh filename=../meshes/Chassis.obj scale=1000
- link RRL1: geometry visual mesh filename=../meshes/RRL1.obj scale=1000
- link RRL2: geometry visual mesh filename=../meshes/RRL2.obj scale=1000
- link RRL3: geometry visual mesh filename=../meshes/RRL3.obj scale=1000
- link RRL4: geometry collision sphere radius=0; visual mesh filename=../meshes/RRL4.stl scale=1000
- link RRS1: geometry visual mesh filename=../meshes/RRS1.obj scale=1000
- link RRS2: geometry visual mesh filename=../meshes/RRS2.obj scale=1000
- link RRS3: geometry visual mesh filename=../meshes/RRS3.obj scale=1000
- link RRS4: geometry visual mesh filename=../meshes/RRS4.obj scale=1000

File: drake/examples/HAMR-URDF/urdf/SLSimple_scaled.urdf (robot description, URDF)
Before this commit: robot SingleLeg, 3 links, 2 joints
Links:
- link Chassis: geometry visual mesh filename=../meshes/Chassis.obj scale=1000
