Commit message: Moved things around so warm starting full model

File: drake/examples/HAMR-URDF/urdf/HAMR_scaledV2.urdf (robot description, URDF)
Before this commit: robot Hamr, 33 links, 32 joints
Links:
- link FLL4: mass 3.0037E-02 -> 3.0948E-02
- link FRL4: mass 3.0037E-02 -> 3.0948E-02
Joints:
- joint FLqfb1: limit (none) -> lower=-pi/6 upper=pi/6
- joint FLqfb3: limit (none) -> lower=-pi/6 upper=pi/6
- joint FLql1: limit (none) -> lower=-pi/6 upper=pi/6
- joint FLql2: limit (none) -> lower=-pi/6 upper=pi/6
- joint FLqs1: limit (none) -> lower=-pi/6 upper=pi/6
- joint FLqs2: limit (none) -> lower=-pi/6 upper=pi/6
- joint FRqfb1: limit (none) -> lower=-pi/6 upper=pi/6
- joint FRqfb3: limit (none) -> lower=-pi/6 upper=pi/6
- joint FRql1: limit (none) -> lower=-pi/6 upper=pi/6
- joint FRql2: limit (none) -> lower=-pi/6 upper=pi/6
- joint FRqs1: limit (none) -> lower=-pi/6 upper=pi/6
- joint FRqs2: limit (none) -> lower=-pi/6 upper=pi/6
- joint RLqfb1: limit (none) -> lower=-pi/6 upper=pi/6
- joint RLqfb3: limit (none) -> lower=-pi/6 upper=pi/6
- joint RLql1: limit (none) -> lower=-pi/6 upper=pi/6
- joint RLql2: limit (none) -> lower=-pi/6 upper=pi/6
- joint RLqs1: limit (none) -> lower=-pi/6 upper=pi/6
- joint RLqs2: limit (none) -> lower=-pi/6 upper=pi/6
- joint RRqfb1: limit (none) -> lower=-pi/6 upper=pi/6
- joint RRqfb3: limit (none) -> lower=-pi/6 upper=pi/6
- joint RRql1: limit (none) -> lower=-pi/6 upper=pi/6
- joint RRql2: limit (none) -> lower=-pi/6 upper=pi/6
- joint RRqs1: limit (none) -> lower=-pi/6 upper=pi/6
- joint RRqs2: limit (none) -> lower=-pi/6 upper=pi/6
