Commit message: renamed some joints

File: drake/examples/Cassie/urdf/cassie_no_loops.urdf (robot description, URDF)
Before this commit: robot cassie, 21 links, 20 joints
Links:
- removed link heel_spring_left
- removed link heel_spring_right
- added link ankle_spring_left, mass 0.126; visual mesh filename=meshes/heel-spring.obj
- added link ankle_spring_right, mass 0.126; visual mesh filename=meshes/heel-spring.obj
Joints:
- removed joint heel_spring_joint_left
- removed joint heel_spring_joint_right
- removed joint knee_left
- removed joint knee_right
- removed joint knee_shin_passive_left
- removed joint knee_shin_passive_right
- removed joint knee_spring_joint_left
- removed joint knee_spring_joint_right
- removed joint shin_tarsus_passive_left
- removed joint shin_tarsus_passive_right
- removed joint toe_crank_left
- removed joint toe_crank_right
- added joint ankle_joint_left: type revolute, parent shin_left, child tarsus_left, origin xyz=0.43476 0.02 0 rpy=0 0 0, axis 0 0 1, limit lower=.8 upper=3
- added joint ankle_joint_right: type revolute, parent shin_right, child tarsus_right, origin xyz=0.43476 0.02 0 rpy=0 0 0, axis 0 0 1, limit lower=.8 upper=3
- added joint ankle_spring_joint_left: type revolute, parent tarsus_left, child ankle_spring_left, origin xyz=-.01269 -.03059 .00092 rpy=-0.0689 -0.0370 2.7208, axis 0 0 1, limit lower=-.1 upper=0.1
- added joint ankle_spring_joint_right: type revolute, parent tarsus_right, child ankle_spring_right, origin xyz=-.01269 -.03059 .00092 rpy=0.0734 0.0269 2.7201, axis 0 0 1, limit lower=-.1 upper=0.1
- added joint knee_joint_left: type revolute, parent knee_left, child shin_left, origin xyz=0.06068 0.04741 0 rpy=0 0 0, axis 0 0 1, limit lower=-.1 upper=0.075
- added joint knee_joint_right: type revolute, parent knee_right, child shin_right, origin xyz=0.06068 0.04741 0 rpy=0 0 0, axis 0 0 1, limit lower=-.1 upper=0.075
- added joint knee_motor_left: type revolute, parent thigh_left, child knee_left, origin xyz=0.12 0 0.045 rpy=0 0 0, axis 0 0 1, limit lower=-2.862 upper=-0.646 effort=50
- added joint knee_motor_right: type revolute, parent thigh_right, child knee_right, origin xyz=0.12 0 -0.045 rpy=0 0 0, axis 0 0 1, limit lower=-2.862 upper=-0.646 effort=50
- added joint knee_spring_left_fixed: type fixed, parent knee_left, child knee_spring_left, origin xyz=0.06068 0.08241 0 rpy=0 0 0
- added joint knee_spring_right_fixed: type fixed, parent knee_right, child knee_spring_right, origin xyz=0.06068 0.08241 0 rpy=0 0 0
- added joint toe_crank_left_fixed: type fixed, parent tarsus_left, child toe_crank_link_left, origin xyz=0.058 -0.034 0.02275 rpy=0 0 0, axis 0 0 1, limit lower=-2.443 upper=-0.524 effort=50
- added joint toe_crank_right_fixed: type fixed, parent tarsus_right, child toe_crank_link_right, origin xyz=0.058 -0.034 -0.02275 rpy=0 0 0, axis 0 0 1, limit lower=-2.443 upper=-0.524 effort=50
