Commit message: fixed renaming bugs

File: drake/examples/Cassie/urdf/cassie.urdf (robot description, URDF)
Before this commit: robot cassie, 33 links, 32 joints
Links:
- removed link achilles_heel_ghost_link_left
- removed link achilles_heel_ghost_link_right
- removed link achilles_rod_left
- removed link achilles_rod_right
- removed link achilles_thigh_ghost_link_left
- removed link achilles_thigh_ghost_link_right
- removed link plantar_crank_ghost_link_left
- removed link plantar_crank_ghost_link_right
- removed link plantar_rod_left
- removed link plantar_rod_right
- removed link plantar_toe_ghost_link_left
- removed link plantar_toe_ghost_link_right
- link toe_left: geometry collision sphere radius=0.0; collision sphere radius=0.0
- link toe_right: geometry collision sphere radius=0.0; collision sphere radius=0.0
Joints:
- removed joint crank_plantar_pitch_passive_left
- removed joint crank_plantar_pitch_passive_right
- removed joint heel_achilles_pitch_passive_left
- removed joint heel_achilles_pitch_passive_right
- removed joint heel_spring_joint_left
- removed joint heel_spring_joint_right
- removed joint knee_left
- removed joint knee_right
- removed joint knee_shin_passive_left
- removed joint knee_shin_passive_right
- removed joint knee_spring_joint_left
- removed joint knee_spring_joint_right
- removed joint shin_tarsus_passive_left
- removed joint shin_tarsus_passive_right
- removed joint thigh_achilles_pitch_passive_left
- removed joint thigh_achilles_pitch_passive_right
- removed joint thigh_achilles_roll_passive_left
- removed joint thigh_achilles_roll_passive_right
- removed joint toe_passive_left
- removed joint toe_passive_right
- removed joint toe_plantar_pitch_passive_left
- removed joint toe_plantar_pitch_passive_right
- removed joint toe_plantar_roll_passive_left
- removed joint toe_plantar_roll_passive_right
- added joint ankle_joint_left: type revolute, parent shin_left, child tarsus_left, origin xyz=0.43476 0.02 0 rpy=0 0 0, axis 0 0 1, limit lower=.8 upper=3
- added joint ankle_joint_right: type revolute, parent shin_right, child tarsus_right, origin xyz=0.43476 0.02 0 rpy=0 0 0, axis 0 0 1, limit lower=.8 upper=3
- added joint ankle_spring_joint_left: type revolute, parent tarsus_left, child heel_spring_left, origin xyz=-.01269 -.03059 .00092 rpy=-0.0689 -0.0370 2.7208, axis 0 0 1, limit lower=-.1 upper=0.1
- added joint ankle_spring_joint_right: type revolute, parent tarsus_right, child heel_spring_right, origin xyz=-.01269 -.03059 .00092 rpy=0.0734 0.0269 2.7201, axis 0 0 1, limit lower=-.1 upper=0.1
- added joint knee_joint_left: type revolute, parent knee_left, child shin_left, origin xyz=0.06068 0.04741 0 rpy=0 0 0, axis 0 0 1, limit lower=-.1 upper=0.075
- added joint knee_joint_right: type revolute, parent knee_right, child shin_right, origin xyz=0.06068 0.04741 0 rpy=0 0 0, axis 0 0 1, limit lower=-.1 upper=0.075
- added joint knee_motor_left: type revolute, parent thigh_left, child knee_left, origin xyz=0.12 0 0.045 rpy=0 0 0, axis 0 0 1, limit lower=-2.862 upper=-0.646 effort=50
- added joint knee_motor_right: type revolute, parent thigh_right, child knee_right, origin xyz=0.12 0 -0.045 rpy=0 0 0, axis 0 0 1, limit lower=-2.862 upper=-0.646 effort=50
- added joint knee_spring_left_fixed: type fixed, parent knee_left, child knee_spring_left, origin xyz=0.06068 0.08241 0 rpy=0 0 0
- added joint knee_spring_right_fixed: type fixed, parent knee_right, child knee_spring_right, origin xyz=0.06068 0.08241 0 rpy=0 0 0
- added joint toe_left: type revolute, parent tarsus_left, child toe_left, origin xyz=0.408 -0.040 0 rpy=0 0 0, axis 0 0 1, limit lower=-2.443 upper=-0.524 effort=50
- added joint toe_right: type revolute, parent tarsus_right, child toe_right, origin xyz=0.408 -0.040 0 rpy=0 0 0, axis 0 0 1, limit lower=-2.443 upper=-0.524 effort=50
- joint toe_crank_left: type revolute -> fixed
- joint toe_crank_right: type revolute -> fixed

File: drake/examples/Cassie/urdf/old/cassie.urdf (robot description, URDF)
Before this commit: robot cassie, 21 links, 20 joints
Links:
- removed link ankle_spring_left
- removed link ankle_spring_right
- added link achilles_heel_ghost_link_left, mass 0.0001
- added link achilles_heel_ghost_link_right, mass 0.0001
- added link achilles_rod_left, mass 0.157; visual mesh filename=meshes/achilles-rod.obj
- added link achilles_rod_right, mass 0.157; visual mesh filename=meshes/achilles-rod.obj
- added link achilles_thigh_ghost_link_left, mass 0.0001
- added link achilles_thigh_ghost_link_right, mass 0.0001
- added link heel_spring_left, mass 0.126; visual mesh filename=meshes/heel-spring.obj
- added link heel_spring_right, mass 0.126; visual mesh filename=meshes/heel-spring.obj
- added link plantar_crank_ghost_link_left, mass 0.0001
- added link plantar_crank_ghost_link_right, mass 0.0001
- added link plantar_rod_left, mass 0.119; visual mesh filename=meshes/plantar-rod.obj
- added link plantar_rod_right, mass 0.119; visual mesh filename=meshes/plantar-rod.obj
- added link plantar_toe_ghost_link_left, mass 0.0001
- added link plantar_toe_ghost_link_right, mass 0.0001
- link toe_left: geometry visual mesh filename=meshes/toe.obj
- link toe_right: geometry visual mesh filename=meshes/toe-r.obj
Joints:
- removed joint ankle_joint_left
- removed joint ankle_joint_right
- removed joint ankle_spring_joint_left
- removed joint ankle_spring_joint_right
- removed joint knee_joint_left
- removed joint knee_joint_right
- removed joint knee_motor_left
- removed joint knee_motor_right
- removed joint knee_spring_left_fixed
- removed joint knee_spring_right_fixed
- removed joint toe_crank_left_fixed
- removed joint toe_crank_right_fixed
- removed joint toe_left
- removed joint toe_right
- added joint crank_plantar_pitch_passive_left: type continuous, parent toe_crank_link_left, child plantar_crank_ghost_link_left, origin xyz=0.055 0 -0.00791 rpy=0 0 0, axis 0 0 1
- added joint crank_plantar_pitch_passive_right: type continuous, parent toe_crank_link_right, child plantar_crank_ghost_link_right, origin xyz=0.055 0 0.00791 rpy=0 0 0, axis 0 0 1
- added joint heel_achilles_pitch_passive_left: type revolute, parent heel_spring_left, child achilles_heel_ghost_link_left, origin xyz=0.11877 -0.01 0 rpy=0 0 0, axis 0 0 1, limit lower=0.6 upper=2.9
- added joint heel_achilles_pitch_passive_right: type revolute, parent heel_spring_right, child achilles_heel_ghost_link_right, origin xyz=0.11877 -0.01 0 rpy=0 0 0, axis 0 0 1, limit lower=0.6 upper=2.9
- added joint heel_spring_joint_left: type fixed, parent tarsus_left, child heel_spring_left, origin xyz=-.01269 -.03059 .00092 rpy=-0.0689 -0.0370 2.7208, axis 0 0 1, limit lower=-.1 upper=0.1
- added joint heel_spring_joint_right: type fixed, parent tarsus_right, child heel_spring_right, origin xyz=-.01269 -.03059 .00092 rpy=0.0734 0.0269 2.7201, axis 0 0 1, limit lower=-.1 upper=0.1
- added joint knee_left: type revolute, parent thigh_left, child knee_left, origin xyz=0.12 0 0.045 rpy=0 0 0, axis 0 0 1, limit lower=-2.862 upper=-0.646 effort=50
- added joint knee_right: type revolute, parent thigh_right, child knee_right, origin xyz=0.12 0 -0.045 rpy=0 0 0, axis 0 0 1, limit lower=-2.862 upper=-0.646 effort=50
- added joint knee_shin_passive_left: type fixed, parent knee_left, child shin_left, origin xyz=0.06068 0.04741 0 rpy=0 0 0, axis 0 0 1, limit lower=-.1 upper=0.075
- added joint knee_shin_passive_right: type fixed, parent knee_right, child shin_right, origin xyz=0.06068 0.04741 0 rpy=0 0 0, axis 0 0 1, limit lower=-.1 upper=0.075
- added joint knee_spring_joint_left: type fixed, parent knee_left, child knee_spring_left, origin xyz=0.06068 0.08241 0 rpy=0 0 0
- added joint knee_spring_joint_right: type fixed, parent knee_right, child knee_spring_right, origin xyz=0.06068 0.08241 0 rpy=0 0 0
- added joint shin_tarsus_passive_left: type revolute, parent shin_left, child tarsus_left, origin xyz=0.43476 0.02 0 rpy=0 0 0, axis 0 0 1, limit lower=.8 upper=3
- added joint shin_tarsus_passive_right: type revolute, parent shin_right, child tarsus_right, origin xyz=0.43476 0.02 0 rpy=0 0 0, axis 0 0 1, limit lower=.8 upper=3
- added joint thigh_achilles_pitch_passive_left: type revolute, parent thigh_left, child achilles_thigh_ghost_link_left, origin xyz=0 0 0.045 rpy=0 0 0, axis 0 0 1, limit lower=-2.75 upper=-0.5
- added joint thigh_achilles_pitch_passive_right: type revolute, parent thigh_right, child achilles_thigh_ghost_link_right, origin xyz=0 0 -0.045 rpy=0 0 0, axis 0 0 1, limit lower=-2.75 upper=-0.5
- added joint thigh_achilles_roll_passive_left: type revolute, parent achilles_thigh_ghost_link_left, child achilles_rod_left, origin xyz=0 0 0 rpy=0 0 0, axis 0 1 0, limit lower=-.05 upper=0.05
- added joint thigh_achilles_roll_passive_right: type revolute, parent achilles_thigh_ghost_link_right, child achilles_rod_right, origin xyz=0 0 0 rpy=0 0 0, axis 0 1 0, limit lower=-.05 upper=0.05
- added joint toe_crank_left: type revolute, parent tarsus_left, child toe_crank_link_left, origin xyz=0.058 -0.034 0.02275 rpy=0 0 0, axis 0 0 1, limit lower=-2.443 upper=-0.524 effort=50
- added joint toe_crank_right: type revolute, parent tarsus_right, child toe_crank_link_right, origin xyz=0.058 -0.034 -0.02275 rpy=0 0 0, axis 0 0 1, limit lower=-2.443 upper=-0.524 effort=50
- added joint toe_passive_left: type revolute, parent tarsus_left, child toe_left, origin xyz=0.408 -0.040 0 rpy=0 0 0, axis 0 0 1, limit lower=-2.443 upper=-0.524
- added joint toe_passive_right: type revolute, parent tarsus_right, child toe_right, origin xyz=0.408 -0.040 0 rpy=0 0 0, axis 0 0 1, limit lower=-2.443 upper=-0.524
- added joint toe_plantar_pitch_passive_left: type revolute, parent toe_left, child plantar_toe_ghost_link_left, origin xyz=0.055 0 0.00776 rpy=0 0 0, axis 0 0 1, limit lower=-2.65 upper=-0.6
- added joint toe_plantar_pitch_passive_right: type revolute, parent toe_right, child plantar_toe_ghost_link_right, origin xyz=0.055 0 -0.00776 rpy=0 0 0, axis 0 0 1, limit lower=-2.65 upper=-0.6
- added joint toe_plantar_roll_passive_left: type revolute, parent plantar_toe_ghost_link_left, child plantar_rod_left, origin xyz=0 0 0 rpy=0 0 0, axis 0 1 0, limit lower=-.1 upper=0.1
- added joint toe_plantar_roll_passive_right: type revolute, parent plantar_toe_ghost_link_right, child plantar_rod_right, origin xyz=0 0 0 rpy=0 0 0, axis 0 1 0, limit lower=-.1 upper=0.1

Commit message: Update urdf to match agility

File: drake/examples/Cassie/urdf/cassie.urdf (robot description, URDF)
Before this commit: robot cassie, 21 links, 20 joints
Links:
- link heel_spring_left: mass 0.126 -> 0.1259
- link heel_spring_right: mass 0.126 -> 0.1259
- link hip_left: mass 1.17 -> 1.171; geometry visual mesh filename=meshes/agility/left_hip.obj
- link hip_right: mass 1.17 -> 1.171; geometry visual mesh filename=meshes/agility/right_hip.obj
- link knee_left: mass 0.758 -> 0.7578
- link knee_right: mass 0.758 -> 0.7578
- link knee_spring_left: mass 0.186 -> 0.1864
- link knee_spring_right: mass 0.186 -> 0.1864
- link shin_left: mass 0.577 -> 0.5771; geometry visual mesh filename=meshes/agility/left_shin.obj
- link shin_right: mass 0.577 -> 0.5771; geometry visual mesh filename=meshes/agility/right_shin.obj
- link thigh_left: geometry visual mesh filename=meshes/agility/left_thigh.obj
- link thigh_right: geometry visual mesh filename=meshes/agility/right_thigh.obj
- link toe_left: mass 0.150 -> 0.1498; geometry collision sphere radius=0.0; collision sphere radius=0.0
- link toe_right: mass 0.150 -> 0.1498; geometry collision sphere radius=0.0; collision sphere radius=0.0
- link yaw_left: geometry visual mesh filename=meshes/agility/left_yaw.obj
- link yaw_right: geometry visual mesh filename=meshes/agility/right_yaw.obj
Joints:
- joint ankle_spring_joint_left: origin xyz=-.01269 -.03059 .00092 rpy=-0.0689 -0.0370 2.7208 -> xyz=-.01269 -.03059 .00092 rpy=0.0780 0.00549 2.7192
- joint ankle_spring_joint_right: origin xyz=-.01269 -.03059 .00092 rpy=0.0734 0.0269 2.7201 -> xyz=-.01269 -.03059 -.00092 rpy=-0.0780 -0.00549 2.7192
- joint knee_motor_left: origin xyz=0.12 0 0.045 rpy=0 0 0 -> xyz=0.12 0 0.0045 rpy=0 0 0
- joint knee_motor_right: origin xyz=0.12 0 -0.045 rpy=0 0 0 -> xyz=0.12 0 -0.0045 rpy=0 0 0
