Commit message: pipeline for fitting working

File: drake/examples/HAMR-URDF/dev/SimpleHAMR/urdf/SLSimple_scaled.urdf (robot description, URDF)
Before this commit: robot SingleLeg, 3 links, 2 joints
Links:
- link Chassis: geometry visual mesh filename=../../../meshes/Chassis.obj scale=1000
Joints:
- joint FL_lift: child FL1 -> FL2; origin xyz=12.75300579825,  9.91, 0.46 rpy=0 0 0 -> xyz=0 0 0 rpy=0 0 0; parent Chassis -> FL1
- joint FL_swing: child FL2 -> FL1; origin xyz=0 0 0 rpy=0 0 0 -> xyz=12.75300579825,  9.91, 0.46 rpy=0 0 0; parent FL1 -> Chassis
