Commit message: working traj_opt

File: drake/examples/HAMR-URDF/dev/SimpleHAMR/urdf/FL_scaled.urdf (robot description, URDF)
Before this commit: robot Hamr, 10 links, 9 joints
Links:
- removed link FLLeg
- link Chassis: mass 1.15747214880841 ->  1.2066
- link FLL4: mass 1.3954E-02 -> 3.0037E-02; geometry collision sphere radius=0; visual mesh filename=../meshes/FLL4.stl scale=1000
Joints:
- removed joint FLLegJoint
- joint FLqfb1: limit (none) -> lower=-pi/3 upper=pi/3
- joint FLqfb3: limit (none) -> lower=-pi/4 upper=pi/4
- joint FLql1: limit (none) -> lower=-pi/3 upper=pi/3
- joint FLql2: limit (none) -> lower=-pi/3 upper=pi/3
- joint FLqs1: limit (none) -> lower=-pi/3 upper=pi/3
- joint FLqs2: limit (none) -> lower=-pi/3 upper=pi/3

File: drake/examples/HAMR-URDF/dev/SimpleHAMR/urdf/FR_scaled.urdf (robot description, URDF)
Before this commit: robot SingleLeg, 9 links, 8 joints
Links:
- removed link FLL1
- removed link FLL2
- removed link FLL3
- removed link FLL4
- removed link FLS1
- removed link FLS2
- removed link FLS3
- removed link FLS4
- added link FRL1, mass 4.5174E-03; visual mesh filename=../meshes/FRL1.obj scale=1000
- added link FRL2, mass 1.6211E-03; visual mesh filename=../meshes/FRL2.obj scale=1000
- added link FRL3, mass 4.2308E-03; visual mesh filename=../meshes/FRL3.obj scale=1000
- added link FRL4, mass 3.0037E-02; collision sphere radius=0; visual mesh filename=../meshes/FRL4.obj scale=1000
- added link FRS1, mass 8.9854E-04; visual mesh filename=../meshes/FRS1.obj scale=1000
- added link FRS2, mass 7.2648E-03; visual mesh filename=../meshes/FRS2.obj scale=1000
- added link FRS3, mass 3.889E-03; visual mesh filename=../meshes/FRS3.obj scale=1000
- added link FRS4, mass 1.4269E-02; visual mesh filename=../meshes/FRS4.obj scale=1000
Joints:
- removed joint FLqfb1
- removed joint FLqfb3
- removed joint FLql1
- removed joint FLql2
- removed joint FLqlact
- removed joint FLqs1
- removed joint FLqs2
- removed joint FLqsact
- added joint FRqfb1: type revolute, parent FRS3, child FRS4, origin xyz=1.52236486487 -0.12 -1.25 rpy=0 0 0, axis 1 0 0
- added joint FRqfb3: type revolute, parent FRL3, child FRL4, origin xyz=2.25 -0.12 -1.07 rpy=0 0 0, axis 0 0 1
- added joint FRql1: type revolute, parent FRL1, child FRL2, origin xyz=0 -4.57322017852 0.38168853124 rpy=0 0 0, axis 1 0 0
- added joint FRql2: type revolute, parent FRL2, child FRL3, origin xyz=0 -1.945 0 rpy=0 0 0, axis 1 0 0
- added joint FRqlact: type prismatic, parent Chassis, child FRL1, origin xyz=10.504659815390 -3.151779821480 -0.501688531240 rpy=0 0 0, axis 0 1 0, limit lower=-0.3 upper=0.3
- added joint FRqs1: type revolute, parent FRS1, child FRS2, origin xyz=0 -0.77116874934 0.12648211488 rpy=0 0 0, axis 0 0 1
- added joint FRqs2: type revolute, parent FRS2, child FRS3, origin xyz=0 -7.44214712409 2.06176831433 rpy=0 0 0, axis 0 0 1
- added joint FRqsact: type prismatic, parent Chassis, child FRS1, origin xyz=13.284659815390 -1.456684126580 -0.478250429210 rpy=0 0 0, axis 0 1 0, limit lower=-0.3 upper=0.3

File: drake/examples/HAMR-URDF/dev/SimpleHAMR/urdf/HAMRSimple_scaled.urdf (robot description, URDF)
Before this commit: robot Hamr, 9 links, 8 joints
Joints:
- joint FL_lift: limit lower=0.1259 upper=0.9113 -> lower=0.1695 upper=0.8677
- joint FL_swing: limit lower=-pi/6 upper=pi/6 -> lower=-pi/9 upper=pi/9
- joint FR_lift: limit lower=-0.9113 upper=-0.1259 -> lower=-0.8677 upper=-0.1695
- joint FR_swing: limit lower=-pi/6 upper=pi/6 -> lower=-pi/9 upper=pi/9
- joint RL_lift: limit lower=0.1259 upper=0.9113 -> lower=0.1695 upper=0.8677
- joint RL_swing: limit lower=-pi/6 upper=pi/6 -> lower=-pi/9 upper=pi/9
- joint RR_lift: limit lower=-0.9113 upper=-0.1259 -> lower=-0.8677 upper=-0.1695
- joint RR_swing: limit lower=-pi/6 upper=pi/6 -> lower=-pi/9 upper=pi/9

File: drake/examples/HAMR-URDF/urdf/HAMR_scaled.urdf (robot description, URDF)
Before this commit: robot Hamr, 37 links, 36 joints
Links:
- removed link RLLeg
- link RLL4: mass 1.3954E-02 -> 3.0948E-02; geometry collision sphere radius=0; visual mesh filename=../meshes/RLL4.stl scale=1000
Joints:
- removed joint RLLegJoint

File: drake/examples/HAMR-URDF/urdf/HAMR_scaledV2.urdf (robot description, URDF)
Before this commit: robot Hamr, 37 links, 36 joints
Links:
- removed link FLLeg
- removed link FRLeg
- removed link RLLeg
- removed link RRLeg
- link Chassis: mass 1.15747214880841 ->  1.2066
- link FLL4: mass 1.3954E-02 -> 3.0037E-02; geometry collision sphere radius=0; visual mesh filename=../meshes/FLL4.stl scale=1000
- link FRL4: mass 1.3954E-02 -> 3.0037E-02; geometry collision sphere radius=0; visual mesh filename=../meshes/FRL4.obj scale=1000
- link RLL4: mass 1.3954E-02 -> 3.0948E-02; geometry collision sphere radius=0; visual mesh filename=../meshes/RLL4.stl scale=1000
- link RRL4: mass 1.3954E-02 -> 3.0948E-02; geometry collision sphere radius=0; visual mesh filename=../meshes/RRL4.stl scale=1000
Joints:
- removed joint FLLegJoint
- removed joint FRLegJoint
- removed joint RLLegJoint
- removed joint RRLegJoint

Commit message: working on reduced order model

File: drake/examples/HAMR-URDF/dev/SimpleHAMR/urdf/FL_scaled.urdf (robot description, URDF)
Before this commit: robot FrontLeftSingleLeg, 9 links, 8 joints
Links:
- link Chassis: geometry visual mesh filename=../../../meshes/Chassis.obj scale=1000
- link FLL1: geometry visual mesh filename=../../../meshes/FLL1.obj scale=1000
- link FLL2: geometry visual mesh filename=../../../meshes/FLL2.obj scale=1000
- link FLL3: geometry visual mesh filename=../../../meshes/FLL3.obj scale=1000
- link FLL4: geometry collision sphere radius=0; visual mesh filename=../../../meshes/FLL4.obj scale=1000
- link FLS1: geometry visual mesh filename=../../../meshes/FLS1.obj scale=1000
- link FLS2: geometry visual mesh filename=../../../meshes/FLS2.obj scale=1000
- link FLS3: geometry visual mesh filename=../../../meshes/FLS3.obj scale=1000
- link FLS4: geometry visual mesh filename=../../../meshes/FLS4.obj scale=1000

File: drake/examples/HAMR-URDF/dev/SimpleHAMR/urdf/FR_scaled.urdf (robot description, URDF)
Before this commit: robot FrontRightSingleLeg, 9 links, 8 joints
Links:
- link Chassis: geometry visual mesh filename=../../../meshes/Chassis.obj scale=1000
- link FRL1: geometry visual mesh filename=../../../meshes/FRL1.obj scale=1000
- link FRL2: geometry visual mesh filename=../../../meshes/FRL2.obj scale=1000
- link FRL3: geometry visual mesh filename=../../../meshes/FRL3.obj scale=1000
- link FRL4: geometry collision sphere radius=0; visual mesh filename=../../../meshes/FRL4.obj scale=1000
- link FRS1: geometry visual mesh filename=../../../meshes/FRS1.obj scale=1000
- link FRS2: geometry visual mesh filename=../../../meshes/FRS2.obj scale=1000
- link FRS3: geometry visual mesh filename=../../../meshes/FRS3.obj scale=1000
- link FRS4: geometry visual mesh filename=../../../meshes/FRS4.obj scale=1000

File: drake/examples/HAMR-URDF/dev/SimpleHAMR/urdf/HAMRSimple_scaled.urdf (robot description, URDF)
Before this commit: robot Hamr, 9 links, 8 joints
Links:
- link Chassis: geometry visual mesh filename=../../../meshes/Chassis.obj scale=1000
- link FL2: geometry collision sphere radius=0; visual cylinder length=14.988382167532292 radius=0.5
- link FR2: geometry collision sphere radius=0; visual cylinder length=14.988382167532292 radius=0.5
- link RL2: geometry collision sphere radius=0; visual cylinder length=14.988382167532292 radius=0.5
- link RR2: geometry collision sphere radius=0; visual cylinder length=14.988382167532292 radius=0.5
Joints:
- joint FL_lift: origin xyz=12.75300579825,  9.91, 0.46 rpy=0 0 0 -> xyz=12.754659815389999,  9.91, 0.46 rpy=0 0 0
- joint FR_lift: origin xyz=12.75300579825, -9.91, 0.46 rpy=0 0 0 -> xyz=12.754659815389999, -9.91, 0.46 rpy=0 0 0
- joint RL_lift: origin xyz=-12.75300579825,  9.91, 0.46 rpy=0 0 0 -> xyz=-12.754659815389999,  9.91, 0.46 rpy=0 0 0
- joint RR_lift: origin xyz=-12.75300579825, -9.91, 0.46 rpy=0 0 0 -> xyz=-12.754659815389999, -9.91, 0.46 rpy=0 0 0

File: drake/examples/HAMR-URDF/dev/SimpleHAMR/urdf/RL_scaled.urdf (robot description, URDF)
Before this commit: robot RearLeftSingleLeg, 9 links, 8 joints
Links:
- link Chassis: geometry visual mesh filename=../../../meshes/Chassis.obj scale=1000
- link RLL1: geometry visual mesh filename=../../../meshes/RLL1.obj scale=1000
- link RLL2: geometry visual mesh filename=../../../meshes/RLL2.obj scale=1000
- link RLL3: geometry visual mesh filename=../../../meshes/RLL3.obj scale=1000
- link RLL4: geometry collision sphere radius=0; visual mesh filename=../../../meshes/RLL4.obj scale=1000
- link RLS1: geometry visual mesh filename=../../../meshes/RLS1.obj scale=1000
- link RLS2: geometry visual mesh filename=../../../meshes/RLS2.obj scale=1000
- link RLS3: geometry visual mesh filename=../../../meshes/RLS3.obj scale=1000
- link RLS4: geometry visual mesh filename=../../../meshes/RLS4.obj scale=1000

File: drake/examples/HAMR-URDF/dev/SimpleHAMR/urdf/RR_scaled.urdf (robot description, URDF)
Before this commit: robot RearRightSingleLeg, 9 links, 8 joints
Links:
- link Chassis: geometry visual mesh filename=../../../meshes/Chassis.obj scale=1000
- link RRL1: geometry visual mesh filename=../../../meshes/RRL1.obj scale=1000
- link RRL2: geometry visual mesh filename=../../../meshes/RRL2.obj scale=1000
- link RRL3: geometry visual mesh filename=../../../meshes/RRL3.obj scale=1000
- link RRL4: geometry collision sphere radius=0; visual mesh filename=../../../meshes/RRL4.stl scale=1000
- link RRS1: geometry visual mesh filename=../../../meshes/RRS1.obj scale=1000
- link RRS2: geometry visual mesh filename=../../../meshes/RRS2.obj scale=1000
- link RRS3: geometry visual mesh filename=../../../meshes/RRS3.obj scale=1000
- link RRS4: geometry visual mesh filename=../../../meshes/RRS4.obj scale=1000

Commit message: Working traj-opt pipeline
ignoring .mat files in HAMR-URDF folder

File: drake/examples/HAMR-URDF/dev/SimpleHAMR/urdf/FL_scaled.urdf (robot description, URDF)
Before this commit: robot FrontLeftSingleLeg, 9 links, 8 joints
Joints:
- joint FLqfb1: limit lower=-pi/3 upper=pi/3 -> lower=-pi/9 upper=pi/9
- joint FLqfb3: limit lower=-pi/4 upper=pi/4 -> lower=-pi/9 upper=pi/9
- joint FLql1: limit lower=-pi/3 upper=pi/3 -> lower=-pi/9 upper=pi/9
- joint FLql2: limit lower=-pi/3 upper=pi/3 -> lower=-pi/9 upper=pi/9
- joint FLqlact: limit lower=-0.3 upper=0.3 -> lower=-0.2 upper=0.2
- joint FLqs1: limit lower=-pi/3 upper=pi/3 -> lower=-pi/9 upper=pi/9
- joint FLqs2: limit lower=-pi/3 upper=pi/3 -> lower=-pi/9 upper=pi/9
- joint FLqsact: limit lower=-0.3 upper=0.3 -> lower=-0.2 upper=0.2

File: drake/examples/HAMR-URDF/dev/SimpleHAMR/urdf/FR_scaled.urdf (robot description, URDF)
Before this commit: robot FrontRightSingleLeg, 9 links, 8 joints
Joints:
- joint FRqfb1: limit (none) -> lower=-pi/9 upper=pi/9
- joint FRqfb3: limit (none) -> lower=-pi/9 upper=pi/9
- joint FRql1: limit (none) -> lower=-pi/9 upper=pi/9
- joint FRql2: limit (none) -> lower=-pi/9 upper=pi/9
- joint FRqlact: limit lower=-0.3 upper=0.3 -> lower=-0.2 upper=0.2
- joint FRqs1: limit (none) -> lower=-pi/9 upper=pi/9
- joint FRqs2: limit (none) -> lower=-pi/9 upper=pi/9
- joint FRqsact: limit lower=-0.3 upper=0.3 -> lower=-0.2 upper=0.2

File: drake/examples/HAMR-URDF/dev/SimpleHAMR/urdf/HAMRSimple_scaled.urdf (robot description, URDF)
Before this commit: robot Hamr, 9 links, 8 joints
Joints:
- joint FL_lift: child FL1 -> FL2; origin xyz=12.754659815389999,  9.91, 0.46 rpy=0 0 0 -> xyz=0 0 0 rpy=0 0 0; parent Chassis -> FL1
- joint FL_swing: child FL2 -> FL1; origin xyz=0 0 0 rpy=0 0 0 -> xyz=12.754659815389999,  9.91, 0.46 rpy=0 0 0; parent FL1 -> Chassis
- joint FR_lift: child FR1 -> FR2; origin xyz=12.754659815389999, -9.91, 0.46 rpy=0 0 0 -> xyz=0 0 0 rpy=0 0 0; parent Chassis -> FR1
- joint FR_swing: child FR2 -> FR1; origin xyz=0 0 0 rpy=0 0 0 -> xyz=12.754659815389999, -9.91, 0.46 rpy=0 0 0; parent FR1 -> Chassis
- joint RL_lift: child RL1 -> RL2; origin xyz=-12.754659815389999,  9.91, 0.46 rpy=0 0 0 -> xyz=0 0 0 rpy=0 0 0; parent Chassis -> RL1
- joint RL_swing: child RL2 -> RL1; origin xyz=0 0 0 rpy=0 0 0 -> xyz=-12.754659815389999,  9.91, 0.46 rpy=0 0 0; parent RL1 -> Chassis
- joint RR_lift: child RR1 -> RR2; origin xyz=-12.754659815389999, -9.91, 0.46 rpy=0 0 0 -> xyz=0 0 0 rpy=0 0 0; parent Chassis -> RR1
- joint RR_swing: child RR2 -> RR1; origin xyz=0 0 0 rpy=0 0 0 -> xyz=-12.754659815389999, -9.91, 0.46 rpy=0 0 0; parent RR1 -> Chassis

File: drake/examples/HAMR-URDF/dev/SimpleHAMR/urdf/RL_scaled.urdf (robot description, URDF)
Before this commit: robot RearLeftSingleLeg, 9 links, 8 joints
Joints:
- joint RLqfb1: limit (none) -> lower=-pi/9 upper=pi/9
- joint RLqfb3: limit (none) -> lower=-pi/9 upper=pi/9
- joint RLql1: limit (none) -> lower=-pi/9 upper=pi/9
- joint RLql2: limit (none) -> lower=-pi/9 upper=pi/9
- joint RLqs1: limit (none) -> lower=-pi/9 upper=pi/9
- joint RLqs2: limit (none) -> lower=-pi/9 upper=pi/9
- joint RLqsact: limit lower=-0.3 upper=0.3 -> lower=-0.2 upper=0.2

File: drake/examples/HAMR-URDF/dev/SimpleHAMR/urdf/RR_scaled.urdf (robot description, URDF)
Before this commit: robot RearRightSingleLeg, 9 links, 8 joints
Joints:
- joint RRqfb1: limit (none) -> lower=-pi/9 upper=pi/9
- joint RRqfb3: limit (none) -> lower=-pi/9 upper=pi/9
- joint RRql1: limit (none) -> lower=-pi/9 upper=pi/9
- joint RRql2: limit (none) -> lower=-pi/9 upper=pi/9
- joint RRqlact: limit lower=-0.3 upper=0.3 -> lower=-0.2 upper=0.2
- joint RRqs1: limit (none) -> lower=-pi/9 upper=pi/9
- joint RRqs2: limit (none) -> lower=-pi/9 upper=pi/9
- joint RRqsact: limit lower=-0.3 upper=0.3 -> lower=-0.2 upper=0.2

File: drake/examples/HAMR-URDF/dev/SimpleHAMR/urdf/SLSimple_scaled.urdf (robot description, URDF)
Before this commit: robot SingleLeg, 3 links, 2 joints
Links:
- removed link FL1
- removed link FL2
- added link L1, mass 0.0001; visual sphere radius=0.5
- added link L2, mass 0.0676; collision sphere radius=0; visual cylinder length=14.97 radius=0.5
Joints:
- removed joint FL_lift
- removed joint FL_swing
- added joint lift: type continuous, parent L1, child L2, origin xyz=0 0 0 rpy=0 0 0, axis 1 0 0, limit lower=0.1695 upper=0.8677
- added joint swing: type continuous, parent Chassis, child L1, origin xyz=12.75300579825,  9.91, 0.46 rpy=0 0 0, axis 0 1 0, limit lower=-pi/9 upper=pi/9

File: drake/examples/HAMR-URDF/urdf/HAMR_scaledV2.urdf (robot description, URDF)
Before this commit: robot Hamr, 33 links, 32 joints
Links:
- link FLL4: geometry collision sphere radius=0; visual mesh filename=../meshes/FLL4.obj scale=1000
